File: Hardware/FeriaInternacional2018/Attiny85_Blinking_Led_FIS2018.sch (EAGLE design)
At the start: 31 parts, among them J1 SPI, U1 ATTINY85-20P

Commit message: Add el salvador logo, open hardware, add eschamtic attiny and isp
Parts:
- R2, R3, R4, R5, R6: value 10k -> 330
Changed lines of the file:
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@@
 <part name="D19" library="SparkFun-LED" deviceset="LED" device="3MM" value="RED"/>
 <part name="D20" library="SparkFun-LED" deviceset="LED" device="3MM" value="RED"/>
-<part name="R2" library="SparkFun-Resistors" deviceset="10KOHM" device="-HORIZ-1/4W-1%" value="10k"/>
-<part name="R3" library="SparkFun-Resistors" deviceset="10KOHM" device="-HORIZ-1/4W-1%" value="10k"/>
-<part name="R4" library="SparkFun-Resistors" deviceset="10KOHM" device="-HORIZ-1/4W-1%" value="10k"/>
-<part name="R5" library="SparkFun-Resistors" deviceset="10KOHM" device="-HORIZ-1/4W-1%" value="10k"/>
-<part name="R6" library="SparkFun-Resistors" deviceset="10KOHM" device="-HORIZ-1/4W-1%" value="10k"/>
+<part name="R2" library="SparkFun-Resistors" deviceset="10KOHM" device="-HORIZ-1/4W-1%" value="330"/>
+<part name="R3" library="SparkFun-Resistors" deviceset="10KOHM" device="-HORIZ-1/4W-1%" value="330"/>
+<part name="R4" library="SparkFun-Resistors" deviceset="10KOHM" device="-HORIZ-1/4W-1%" value="330"/>
+<part name="R5" library="SparkFun-Resistors" deviceset="10KOHM" device="-HORIZ-1/4W-1%" value="330"/>
+<part name="R6" library="SparkFun-Resistors" deviceset="10KOHM" device="-HORIZ-1/4W-1%" value="330"/>
 <part name="S1" library="SparkFun-Switches" deviceset="SWITCH-SPDT" device="-SMD-RIGHT-ANGLE" value="SWITCH"/>
 <part name="J1" library="SparkFun-Connectors" deviceset="CONN_03X2" device="POGO_PINS" value="SPI"/>
